Commit message: Added Robotic arm and changed bot model physically

File: src/bme_ros2_navigation/urdf/mogi_bot.urdf (robot description, URDF)
Before this commit: robot mogi_bot, 8 links, 7 joints
Links:
- added link arm_base_link, mass 2; collision cylinder length=0.05 radius=0.15; visual cylinder length=0.05 radius=0.15
- added link end_effector_link, mass 1.0e-03; visual box size=0.01 0.01 0.01
- added link forearm_link, mass 0.2; collision cylinder length=0.25 radius=0.025; visual mesh filename=package://bme_ros2_navigation/meshes/forearm.dae
- added link gripper_base, mass 0.1; collision box size=.05 .1 .01; visual box size=.05 .1 .01
- added link left_finger, mass 0.1; collision box size=.04 .01 .08; visual box size=.04 .01 .08
- added link right_finger, mass 0.1; collision box size=.04 .01 .08; visual box size=.04 .01 .08
- added link shoulder_link, mass 0.5; collision cylinder length=0.05 radius=0.1; visual mesh filename=package://bme_ros2_navigation/meshes/shoulder.dae
- added link upper_arm_link, mass 0.3; collision cylinder length=0.2 radius=0.05; visual mesh filename=package://bme_ros2_navigation/meshes/upper_arm.dae
- added link wrist_link, mass 0.1; collision cylinder length=0.1 radius=0.02; visual mesh filename=package://bme_ros2_navigation/meshes/wrist.dae
- link base_link: geometry collision box size=.4 .3 .1; collision sphere radius=0.0374
- link left_wheel: geometry collision cylinder length=.0375 radius=.075; visual mesh filename=package://bme_ros2_navigation/meshes/wheel.dae scale=0.75 0.75 0.75
- link right_wheel: geometry collision cylinder length=.0375 radius=.075; visual mesh filename=package://bme_ros2_navigation/meshes/wheel.dae scale=0.75 0.75 0.75
Joints:
- added joint arm_base_joint: type fixed, parent base_link, child arm_base_link, origin xyz=0.0 0 0.15 rpy=0 0 0
- added joint elbow_joint: type revolute, parent upper_arm_link, child forearm_link, origin xyz=0.0 0.0 0.2 rpy=0.0 0.0 0.0, axis 0 1 0, limit lower=-2.3562 upper=2.3562 effort=150.0 velocity=3.14
- added joint end_effector_joint: type fixed, parent wrist_link, child end_effector_link, origin xyz=0.0 0.0 0.175 rpy=0 0 0
- added joint gripper_base_joint: type fixed, parent wrist_link, child gripper_base, origin xyz=0.0 0 0.105 rpy=0.0 0 0
- added joint left_finger_joint: type prismatic, parent gripper_base, child left_finger, origin xyz=0.0 0.01 0.045, axis 0 1 0, limit lower=0 upper=0.04 effort=100.0 velocity=4.0
- added joint right_finger_joint: type prismatic, parent gripper_base, child right_finger, origin xyz=0.0 -0.01 0.045, axis 0 -1 0, limit lower=0 upper=0.04 effort=100.0 velocity=4.0
- added joint shoulder_lift_joint: type revolute, parent shoulder_link, child upper_arm_link, origin xyz=0.0 0.0 0.025 rpy=0.0 0.0 0.0, axis 0 1 0, limit lower=-1.5708 upper=1.5708 effort=330.0 velocity=3.14
- added joint shoulder_pan_joint: type revolute, parent arm_base_link, child shoulder_link, origin xyz=0 0 0.05, axis 0 0 1, limit lower=-3.14 upper=3.14 effort=330.0 velocity=3.14
- added joint wrist_joint: type revolute, parent forearm_link, child wrist_link, origin xyz=0.0 0.0 0.25 rpy=0.0 0.0 0.0, axis 0 1 0, limit lower=-2.3562 upper=2.3562 effort=54.0 velocity=3.14
- joint camera_joint: origin xyz=0.225 0 0.075 rpy=0 0 0 -> xyz=0.215 0 0.035 rpy=0 0 0
- joint left_wheel_joint: origin xyz=0 0.15 0 rpy=0 0 0 -> xyz=0 0.18 0 rpy=0 0 0
- joint right_wheel_joint: origin xyz=0 -0.15 0 rpy=0 0 0 -> xyz=0 -0.18 0 rpy=0 0 0
- joint scan_joint: origin xyz=0.0 0 0.15 rpy=0 0 0 -> xyz=0.0 0 0.08 rpy=0 0 0
